File: z-axis-duplicator/rev-1.sch (EAGLE design)
At the start: 18 parts, among them J1 SOLDER-JUMPER, Q1 MMBT3904,215MMBT3904,215, Q2 MMBT3904,215MMBT3904,215, Q3 MMBT3904,215MMBT3904,215

Commit message: Finished schematic
Parts:
- added J2, J3: SOLDER-JUMPER-DUAL, z-axis-duplicator:SOLDER-JUMPER-DUAL
- added J4: JST-PH6, z-axis-duplicator:JST-PH6
Connections:
- new net 1A: A2.1A, J4.P$5, J4.P$6
- new net 1B: J2.2, J3.1, J4.P$4
- new net 2A: J2.1, J3.2, J4.P$3
- new net 2B: A2.2B, J4.P$1, J4.P$2
- new net N$6: A2.1B, J2.C
- new net N$8: A2.2A, J3.C
Other:
- note removed: "TODO"
Changed lines of the file:
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@@
 <part name="GND9" library="z-axis-duplicator" deviceset="GND" device=""/>
 <part name="R8" library="z-axis-duplicator" deviceset="RESISTOR" device="0805" value="20k"/>
+<part name="J2" library="z-axis-duplicator" deviceset="SOLDER-JUMPER-DUAL" device=""/>
+<part name="J3" library="z-axis-duplicator" deviceset="SOLDER-JUMPER-DUAL" device=""/>
+<part name="J4" library="z-axis-duplicator" deviceset="JST-PH6" device="" package3d_urn="urn:adsk.eagle:package:16196389/1"/>
 </parts>
 <sheets>
@@
 <description>Duplicated Driver</description>
 <plain>
-<text x="20.32" y="-2.54" size="1.778" layer="91" rot="R270" align="center">TODO</text>
 </plain>
 <instances>
@@
 <instance part="GND5" gate="1" x="12.7" y="12.7" smashed="yes"/>
 <instance part="GND6" gate="1" x="0" y="-20.32" smashed="yes"/>
+<instance part="J2" gate="G$1" x="35.56" y="2.54" smashed="yes" rot="R270">
+<attribute name="NAME" x="36.5125" y="2.54" size="1.016" layer="95" rot="R270" align="bottom-center"/>
+</instance>
+<instance part="J3" gate="G$1" x="35.56" y="-7.62" smashed="yes" rot="R270">
+<attribute name="NAME" x="36.5125" y="-7.62" size="1.016" layer="95" rot="R270" align="bottom-center"/>
+</instance>
+<instance part="J4" gate="G$1" x="55.88" y="-10.16" smashed="yes">
+<attribute name="NAME" x="55.88" y="7.62" size="1.27" layer="95"/>
+</instance>
 </instances>
 <busses>
@@
 </segment>
 </net>
+<net name="1A" class="0">
+<segment>
+<pinref part="A2" gate="G$1" pin="1A"/>
+<wire x1="17.78" y1="0" x2="27.94" y2="0" width="0.1524" layer="91"/>
+<label x="20.32" y="0" size="1.778" layer="95"/>
+</segment>
+<segment>
+<pinref part="J4" gate="G$1" pin="P$6"/>
+<wire x1="58.42" y1="5.08" x2="53.34" y2="5.08" width="0.1524" layer="91"/>
+<wire x1="53.34" y1="5.08" x2="53.34" y2="2.54" width="0.1524" layer="91"/>
+<pinref part="J4" gate="G$1" pin="P$5"/>
+<wire x1="53.34" y1="2.54" x2="58.42" y2="2.54" width="0.1524" layer="91"/>
+<wire x1="53.34" y1="5.08" x2="48.26" y2="5.08" width="0.1524" layer="91"/>
+<junction x="53.34" y="5.08"/>
+<label x="48.26" y="5.08" size="1.778" layer="95"/>
+</segment>
+</net>
+<net name="2B" class="0">
+<segment>
+<pinref part="A2" gate="G$1" pin="2B"/>
+<wire x1="17.78" y1="-7.62" x2="27.94" y2="-7.62" width="0.1524" layer="91"/>
+<label x="20.32" y="-7.62" size="1.778" layer="95"/>
+</segment>
+<segment>
+<pinref part="J4" gate="G$1" pin="P$2"/>
+<wire x1="58.42" y1="-5.08" x2="53.34" y2="-5.08" width="0.1524" layer="91"/>
+<wire x1="53.34" y1="-5.08" x2="53.34" y2="-7.62" width="0.1524" layer="91"/>
+<pinref part="J4" gate="G$1" pin="P$1"/>
+<wire x1="53.34" y1="-7.62" x2="58.42" y2="-7.62" width="0.1524" layer="91"/>
+<wire x1="53.34" y1="-7.62" x2="48.26" y2="-7.62" width="0.1524" layer="91"/>
+<junction x="53.34" y="-7.62"/>
+<label x="48.26" y="-7.62" size="1.778" layer="95"/>
+</segment>
+</net>
+<net name="N$6" class="0">
+<segment>
+<pinref part="A2" gate="G$1" pin="1B"/>
+<wire x1="17.78" y1="-2.54" x2="30.48" y2="-2.54" width="0.1524" layer="91"/>
+<wire x1="30.48" y1="-2.54" x2="30.48" y2="2.54" width="0.1524" layer="91"/>
+<pinref part="J2" gate="G$1" pin="C"/>
+<wire x1="30.48" y1="2.54" x2="33.02" y2="2.54" width="0.1524" layer="91"/>
+</segment>
+</net>
+<net name="N$8" class="0">
+<segment>
+<pinref part="A2" gate="G$1" pin="2A"/>
+<wire x1="17.78" y1="-5.08" x2="30.48" y2="-5.08" width="0.1524" layer="91"/>
+<pinref part="J3" gate="G$1" pin="C"/>
+<wire x1="30.48" y1="-5.08" x2="30.48" y2="-7.62" width="0.1524" layer="91"/>
+<wire x1="30.48" y1="-7.62" x2="33.02" y2="-7.62" width="0.1524" layer="91"/>
+</segment>
+</net>
+<net name="1B" class="0">
+<segment>
+<pinref part="J2" gate="G$1" pin="2"/>
+<pinref part="J3" gate="G$1" pin="1"/>
+<wire x1="35.56" y1="0" x2="35.56" y2="-2.54" width="0.1524" layer="91"/>
+<wire x1="35.56" y1="-2.54" x2="35.56" y2="-5.08" width="0.1524" layer="91"/>
+<wire x1="35.56" y1="-2.54" x2="40.64" y2="-2.54" width="0.1524" layer="91"/>
+<junction x="35.56" y="-2.54"/>
+<label x="38.1" y="-2.54" size="1.778" layer="95"/>
+</segment>
+<segment>
+<pinref part="J4" gate="G$1" pin="P$4"/>
+<wire x1="58.42" y1="0" x2="48.26" y2="0" width="0.1524" layer="91"/>
+<label x="48.26" y="0" size="1.778" layer="95"/>
+</segment>
+</net>
+<net name="2A" class="0">
+<segment>
+<pinref part="J3" gate="G$1" pin="2"/>
+<wire x1="35.56" y1="-10.16" x2="35.56" y2="-12.7" width="0.1524" layer="91"/>
+<wire x1="35.56" y1="-12.7" x2="43.18" y2="-12.7" width="0.1524" layer="91"/>
+<wire x1="43.18" y1="-12.7" x2="43.18" y2="7.62" width="0.1524" layer="91"/>
+<wire x1="43.18" y1="7.62" x2="35.56" y2="7.62" width="0.1524" layer="91"/>
+<pinref part="J2" gate="G$1" pin="1"/>
+<wire x1="35.56" y1="7.62" x2="35.56" y2="5.08" width="0.1524" layer="91"/>
+<label x="38.1" y="7.62" size="1.778" layer="95"/>
+</segment>
+<segment>
+<pinref part="J4" gate="G$1" pin="P$3"/>
+<wire x1="58.42" y1="-2.54" x2="48.26" y2="-2.54" width="0.1524" layer="91"/>
+<label x="48.26" y="-2.54" size="1.778" layer="95"/>
+</segment>
+</net>
